File: h743xi-som.kicad_sch (KiCad schematic)
At the start: 3 parts, among them IC1 IS42S16160J-6BLI, IC2 S34ML01G200BHI000, U1 STM32H743XIH6

Commit message: Added my own memory libs, because snapeda or octopart gave me wrong pin library
Parts:
- removed IC1: IS42S16160J-6BLI, IS42S16160J-6BLI:BGA54C80P9X9_800X800X120, symbol IS42S16160J-6BLI:IS42S16160J-6BLI
- removed IC2: S34ML01G200BHI000, S34ML01G200BHI000:BGA63C80P10X12_900X1100X100, symbol S34ML01G200BHI000:S34ML01G200BHI000
- removed unit 1 of U1
- removed unit 3 of U1
Connections:
- no-connect marks 50 -> 10
Other:
- added sheet Memory (memory.kicad_sch)
- added sheet POWER (power.kicad_sch)
